Commit message: gazebo tags for NU ridgeback

File: urdf/nu_ridgeback.gazebo.xacro (robot description, xacro)
@@ -2,5 +2,5 @@
 <robot xmlns:xacro="http://ros.org/wiki/xacro">
   <gazebo reference="mount_link">
-    <material>Gazebo/Red</material>
+    <material>Gazebo/White</material>
   </gazebo>
   <gazebo reference="controller_enclosure">
