Commit message: ridgeback with sawyer mounts and sensors

File: urdf/nu_ridgeback_extras.urdf.xacro (robot description, xacro)
@@ -46,8 +46,8 @@
  </joint>
 <!-- Create a link between the VLP16 mesh and sensor origin -->
- <link name="velodyne" />
+<link name="velodyne_scan"/>
  <joint name="vlp16_mesh_to_vlp16_origin" type="fixed">
    <parent link="velodyne_mesh" />
-   <child link="velodyne" />
+   <child link="velodyne_scan" />
    <origin xyz="0 0 0.195" rpy="0 0 0" />
  </joint>
@@ -66,9 +66,15 @@
  </joint>
 <!-- Create a link between the BB2 mesh and sensor origin -->
- <link name="bumblebee" />
+ <link name="bb2_origin" />
  <joint name="bb2_mesh_to_bb2_origin" type="fixed">
    <parent link="bb2_mesh" />
-   <child link="bumblebee" />
-   <origin xyz="0.001 0 0.07" rpy="0 0 0" />
+   <child link="bb2_origin" />
+   <origin xyz="0.001 0 0.07" rpy="${0} 0 ${-1.5708}" />
+ </joint>
+ <link name="bb2_optical_link" />
+ <joint name="bb2_origin_to_bb2_camera" type="fixed">
+   <parent link="bb2_origin" />
+   <child link="bb2_optical_link" />
+   <origin xyz="0.05 0 0" rpy="${-1.5708} ${0} ${-1.5708}" />
  </joint>
 </robot>

Commit message: sensor suite for NU ridgback

File: urdf/nu_ridgeback_extras.urdf.xacro (robot description, xacro)
@@ -70,5 +70,5 @@
    <parent link="bb2_mesh" />
    <child link="bb2_origin" />
-   <origin xyz="0.001 0 0.07" rpy="${0} 0 ${-1.5708}" />
+   <origin xyz="0.001 0 0.07" rpy="0 0 ${-1.5708}" />
  </joint>
  <link name="bb2_optical_link" />
@@ -76,5 +76,5 @@
    <parent link="bb2_origin" />
    <child link="bb2_optical_link" />
-   <origin xyz="0.05 0 0" rpy="${-1.5708} ${0} ${-1.5708}" />
+   <origin xyz="0.01 0 0" rpy="${-1.5708} 0 ${-1.5708}" />
  </joint>
 </robot>
